File: Hardware/JACR.kicad_pcb (KiCad board)
At the start: 2 copper layers, 100 x 100 mm, 40 parts, among them J1 Barrel_Jack_Switch, J2 JACR CARTRIDGE SLOT, J3 EXP1, J4 EXP2, M1 MountingHole_2.2mm_M2_Pad, M2 MountingHole_2.2mm_M2_Pad, M3 MountingHole_2.2mm_M2_Pad, M4 MountingHole_2.2mm_M2_Pad, Q1 BSS138, Q2 BSS138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

Commit message: Corrected Source and Drain inputs on BSS138 in clock generator circuit
It would seem I have the 3V and 5V flipped and may have been the cause of my clock generator appearing to not work
also made adjustments to some traces
Connections:
- Q1 pad 2: D20 -> /SDA
- Q1 pad 3: /SDA -> D20
- Q2 pad 2: D21 -> /SCL
- Q2 pad 3: /SCL -> D21
Routing:
- net +5V: track 293.6 -> 337.6 mm
- net RST: track 203.8 -> 199.4 mm
- net /SDA: track 5.93 -> 8.94 mm
- net /SCL: track 6.63 -> 9.18 mm
- net D20: track 81.2 -> 82.9 mm
- net +3V3: track 235.8 -> 234.3 mm
- net GND: vias 151 -> 156
